File: SBK6AC/sbk6ac.kicad_pcb (KiCad board)
At the start: 2 copper layers, 98.6 x 99.8 mm, 24 parts, among them IC101 TPIC6C596D, IC102 TPIC6C596D, K101 CONN_31, K102 CONN_31, U101 78L05

Commit message: SBK6AC cleanup
Other:
- net class Default removed
- rule pad_to_mask_clearance: 0.254 -> 0
